File: raspberrypi_isp_tool.sch (EAGLE design)
At the start: 1 part, among them J1 RASPBERRYPI-GPIOPTH

Commit message: More work on breakout utility
Parts:
- added ISP1: AVRISP-6, adafruit:AVRISP-6
- added JP1: (no value), pinhead:PINHD-2X2
- added JP2: (no value), pinhead:PINHD-1X4
Connections:
- new net +3V3: ISP1.VCC, J1.3.3V@1
- new net +5V: J1.5V@2, JP2.1
- new net GND: ISP1.GND, J1.GND@14, J1.GND@20, J1.GND@25, J1.GND@6, J1.GND@9, JP2.2
- new net RX: J1.RXI, JP2.4
- new net TX: J1.TXO, JP2.3
Changed lines of the file:
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@@
 <?xml version="1.0" encoding="utf-8"?>
 <!DOCTYPE eagle SYSTEM "eagle.dtd">
-<eagle version="7.6.0">
+<eagle version="7.5.0">
 <drawing>
 <settings>
@@
 <layer number="230" name="230bmp" color="7" fill="1" visible="yes" active="yes"/>
 <layer number="231" name="231bmp" color="7" fill="1" visible="yes" active="yes"/>
+<layer number="232" name="Eagle3D_PG2" color="7" fill="1" visible="no" active="no"/>
+<layer number="233" name="Eagle3D_PG3" color="7" fill="1" visible="no" active="no"/>
 <layer number="248" name="Housing" color="7" fill="1" visible="yes" active="yes"/>
 <layer number="249" name="Edge" color="7" fill="1" visible="yes" active="yes"/>
@@
 <part name="FRAME1" library="frames" deviceset="FRAME_A_L" device=""/>
 <part name="J1" library="SparkFun-Boards" deviceset="RASPBERRYPI-GPIO" device="PTH"/>
+<part name="ISP1" library="adafruit" deviceset="AVRISP" device="-6"/>
+<part name="JP1" library="pinhead" deviceset="PINHD-2X2" device=""/>
+<part name="JP2" library="pinhead" deviceset="PINHD-1X4" device=""/>
+<part name="P+1" library="supply1" deviceset="+5V" device=""/>
+<part name="P+2" library="supply1" deviceset="+5V" device=""/>
+<part name="+3V1" library="supply1" deviceset="+3V3" device=""/>
+<part name="+3V2" library="supply1" deviceset="+3V3" device=""/>
+<part name="GND1" library="supply1" deviceset="GND" device=""/>
+<part name="GND2" library="supply1" deviceset="GND" device=""/>
+<part name="GND3" library="supply1" deviceset="GND" device=""/>
 </parts>
 <sheets>
@@
 <instance part="FRAME1" gate="G$2" x="152.4" y="-12.7"/>
 <instance part="J1" gate="JP1" x="48.26" y="96.52"/>
+<instance part="ISP1" gate="G$1" x="124.46" y="119.38"/>
+<instance part="JP1" gate="A" x="127" y="139.7"/>
+<instance part="JP2" gate="A" x="129.54" y="78.74"/>
+<instance part="P+1" gate="1" x="22.86" y="127"/>
+<instance part="P+2" gate="1" x="116.84" y="88.9"/>
+<instance part="+3V1" gate="G$1" x="12.7" y="127"/>
+<instance part="+3V2" gate="G$1" x="147.32" y="127"/>
+<instance part="GND1" gate="1" x="20.32" y="66.04"/>
+<instance part="GND2" gate="1" x="106.68" y="76.2"/>
+<instance part="GND3" gate="1" x="147.32" y="109.22"/>
 </instances>
 <busses>
 </busses>
 <nets>
+<net name="TX" class="0">
+<segment>
+<pinref part="JP2" gate="A" pin="3"/>
+<wire x1="119.38" y1="78.74" x2="127" y2="78.74" width="0.1524" layer="91"/>
+<label x="119.38" y="78.74" size="1.778" layer="95"/>
+</segment>
+<segment>
+<pinref part="J1" gate="JP1" pin="TXO"/>
+<wire x1="63.5" y1="114.3" x2="73.66" y2="114.3" width="0.1524" layer="91"/>
+<label x="68.58" y="114.3" size="1.778" layer="95"/>
+</segment>
+</net>
+<net name="RX" class="0">
+<segment>
+<pinref part="JP2" gate="A" pin="4"/>
+<wire x1="119.38" y1="76.2" x2="127" y2="76.2" width="0.1524" layer="91"/>
+<label x="119.38" y="76.2" size="1.778" layer="95"/>
+</segment>
+<segment>
+<pinref part="J1" gate="JP1" pin="RXI"/>
+<wire x1="73.66" y1="111.76" x2="63.5" y2="111.76" width="0.1524" layer="91"/>
+<label x="68.58" y="111.76" size="1.778" layer="95"/>
+</segment>
+</net>
+<net name="GND" class="0">
+<segment>
+<pinref part="GND1" gate="1" pin="GND"/>
+<wire x1="20.32" y1="68.58" x2="20.32" y2="73.66" width="0.1524" layer="91"/>
+<pinref part="J1" gate="JP1" pin="GND@6"/>
+<wire x1="20.32" y1="73.66" x2="20.32" y2="76.2" width="0.1524" layer="91"/>
+<wire x1="20.32" y1="76.2" x2="20.32" y2="78.74" width="0.1524" layer="91"/>
+<wire x1="20.32" y1="78.74" x2="20.32" y2="81.28" width="0.1524" layer="91"/>
+<wire x1="20.32" y1="81.28" x2="20.32" y2="83.82" width="0.1524" layer="91"/>
+<wire x1="20.32" y1="83.82" x2="33.02" y2="83.82" width="0.1524" layer="91"/>
+<pinref part="J1" gate="JP1" pin="GND@9"/>
+<wire x1="33.02" y1="81.28" x2="20.32" y2="81.28" width="0.1524" layer="91"/>
+<junction x="20.32" y="81.28"/>
+<pinref part="J1" gate="JP1" pin="GND@14"/>
+<wire x1="33.02" y1="78.74" x2="20.32" y2="78.74" width="0.1524" layer="91"/>
+<junction x="20.32" y="78.74"/>
+<pinref part="J1" gate="JP1" pin="GND@20"/>
+<wire x1="33.02" y1="76.2" x2="20.32" y2="76.2" width="0.1524" layer="91"/>
+<junction x="20.32" y="76.2"/>
+<pinref part="J1" gate="JP1" pin="GND@25"/>
+<wire x1="33.02" y1="73.66" x2="20.32" y2="73.66" width="0.1524" layer="91"/>
+<junction x="20.32" y="73.66"/>
+</segment>
+<segment>
+<pinref part="ISP1" gate="G$1" pin="GND"/>
+<pinref part="GND3" gate="1" pin="GND"/>
+<wire x1="139.7" y1="116.84" x2="147.32" y2="116.84" width="0.1524" layer="91"/>
+<wire x1="147.32" y1="116.84" x2="147.32" y2="111.76" width="0.1524" layer="91"/>
+</segment>
+<segment>
+<pinref part="GND2" gate="1" pin="GND"/>
+<wire x1="106.68" y1="78.74" x2="106.68" y2="81.28" width="0.1524" layer="91"/>
+<pinref part="JP2" gate="A" pin="2"/>
+<wire x1="106.68" y1="81.28" x2="127" y2="81.28" width="0.1524" layer="91"/>
+</segment>
+</net>
+<net name="+5V" class="0">
+<segment>
+<pinref part="J1" gate="JP1" pin="5V@2"/>
+<pinref part="P+1" gate="1" pin="+5V"/>
+<wire x1="33.02" y1="121.92" x2="22.86" y2="121.92" width="0.1524" layer="91"/>
+<wire x1="22.86" y1="121.92" x2="22.86" y2="124.46" width="0.1524" layer="91"/>
+</segment>
+<segment>
+<pinref part="P+2" gate="1" pin="+5V"/>
+<wire x1="116.84" y1="86.36" x2="116.84" y2="83.82" width="0.1524" layer="91"/>
+<pinref part="JP2" gate="A" pin="1"/>
+<wire x1="116.84" y1="83.82" x2="127" y2="83.82" width="0.1524" layer="91"/>
+</segment>
+</net>
+<net name="+3V3" class="0">
+<segment>
+<pinref part="J1" gate="JP1" pin="3.3V@1"/>
+<pinref part="+3V1" gate="G$1" pin="+3V3"/>
+<wire x1="33.02" y1="116.84" x2="12.7" y2="116.84" width="0.1524" layer="91"/>
+<wire x1="12.7" y1="116.84" x2="12.7" y2="124.46" width="0.1524" layer="91"/>
+</segment>
+<segment>
+<pinref part="ISP1" gate="G$1" pin="VCC"/>
+<pinref part="+3V2" gate="G$1" pin="+3V3"/>
+<wire x1="139.7" y1="121.92" x2="147.32" y2="121.92" width="0.1524" layer="91"/>
+<wire x1="147.32" y1="121.92" x2="147.32" y2="124.46" width="0.1524" layer="91"/>
+</segment>
+</net>
 </nets>
 </sheet>

Commit message: Finished layout for rev a
Parts:
- removed JP1: (no value), pinhead:PINHD-2X2
- added I2C: (no value), SparkFun-Connectors:M02PTH
- added SPI: (no value), SparkFun-Connectors:M05PTH
- renumbered ISP1 to ISP, JP2 to UART
Connections:
- new net CE0: J1.CE0, SPI.2
- new net CE1: J1.CE1, SPI.1
- new net MISO: ISP.MISO, J1.MISO, SPI.4
- new net MOSI: ISP.MOSI, J1.MOSI, SPI.3
- new net RST: ISP.RST, J1.GP22
- new net SCK: ISP.SCK, J1.SCLK, SPI.5
- new net SCL: I2C.1, J1.SCL
- new net SDA: I2C.2, J1.SDA
- net +3V3: now also J1.3.3V@17
Changed lines of the file:
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@@
 <?xml version="1.0" encoding="utf-8"?>
 <!DOCTYPE eagle SYSTEM "eagle.dtd">
-<eagle version="7.5.0">
+<eagle version="7.6.0">
 <drawing>
 <settings>
@@
 <layer number="113" name="IDFDebug" color="7" fill="1" visible="yes" active="yes"/>
 <layer number="114" name="Badge_Outline" color="11" fill="1" visible="no" active="no"/>
+<layer number="115" name="ReferenceISLANDS" color="7" fill="1" visible="yes" active="yes"/>
 <layer number="116" name="Patch_BOT" color="9" fill="4" visible="yes" active="yes"/>
 <layer number="118" name="Rect_Pads" color="7" fill="1" visible="yes" active="yes"/>
@@
 <part name="FRAME1" library="frames" deviceset="FRAME_A_L" device=""/>
 <part name="J1" library="SparkFun-Boards" deviceset="RASPBERRYPI-GPIO" device="PTH"/>
-<part name="ISP1" library="adafruit" deviceset="AVRISP" device="-6"/>
-<part name="JP1" library="pinhead" deviceset="PINHD-2X2" device=""/>
-<part name="JP2" library="pinhead" deviceset="PINHD-1X4" device=""/>
+<part name="ISP" library="adafruit" deviceset="AVRISP" device="-6"/>
+<part name="UART" library="pinhead" deviceset="PINHD-1X4" device=""/>
 <part name="P+1" library="supply1" deviceset="+5V" device=""/>
 <part name="P+2" library="supply1" deviceset="+5V" device=""/>
@@
 <part name="GND2" library="supply1" deviceset="GND" device=""/>
 <part name="GND3" library="supply1" deviceset="GND" device=""/>
+<part name="I2C" library="SparkFun-Connectors" deviceset="M02" device="PTH"/>
+<part name="SPI" library="SparkFun-Connectors" deviceset="M05" device="PTH"/>
 </parts>
 <sheets>
@@
 <instance part="FRAME1" gate="G$2" x="152.4" y="-12.7"/>
 <instance part="J1" gate="JP1" x="48.26" y="96.52"/>
-<instance part="ISP1" gate="G$1" x="124.46" y="119.38"/>
-<instance part="JP1" gate="A" x="127" y="139.7"/>
-<instance part="JP2" gate="A" x="129.54" y="78.74"/>
+<instance part="ISP" gate="G$1" x="124.46" y="119.38"/>
+<instance part="UART" gate="A" x="129.54" y="78.74"/>
 <instance part="P+1" gate="1" x="22.86" y="127"/>
 <instance part="P+2" gate="1" x="116.84" y="88.9"/>
@@
 <instance part="GND2" gate="1" x="106.68" y="76.2"/>
 <instance part="GND3" gate="1" x="147.32" y="109.22"/>
+<instance part="I2C" gate="G$1" x="127" y="147.32"/>
+<instance part="SPI" gate="G$1" x="91.44" y="147.32"/>
 </instances>
 <busses>
@@
 <net name="TX" class="0">
 <segment>
-<pinref part="JP2" gate="A" pin="3"/>
+<pinref part="UART" gate="A" pin="3"/>
 <wire x1="119.38" y1="78.74" x2="127" y2="78.74" width="0.1524" layer="91"/>
 <label x="119.38" y="78.74" size="1.778" layer="95"/>
@@
 <net name="RX" class="0">
 <segment>
-<pinref part="JP2" gate="A" pin="4"/>
+<pinref part="UART" gate="A" pin="4"/>
 <wire x1="119.38" y1="76.2" x2="127" y2="76.2" width="0.1524" layer="91"/>
 <label x="119.38" y="76.2" size="1.778" layer="95"/>
@@
 </segment>
 <segment>
-<pinref part="ISP1" gate="G$1" pin="GND"/>
+<pinref part="ISP" gate="G$1" pin="GND"/>
 <pinref part="GND3" gate="1" pin="GND"/>
 <wire x1="139.7" y1="116.84" x2="147.32" y2="116.84" width="0.1524" layer="91"/>
@@
 <pinref part="GND2" gate="1" pin="GND"/>
 <wire x1="106.68" y1="78.74" x2="106.68" y2="81.28" width="0.1524" layer="91"/>
-<pinref part="JP2" gate="A" pin="2"/>
+<pinref part="UART" gate="A" pin="2"/>
 <wire x1="106.68" y1="81.28" x2="127" y2="81.28" width="0.1524" layer="91"/>
 </segment>
@@
 <pinref part="P+2" gate="1" pin="+5V"/>
 <wire x1="116.84" y1="86.36" x2="116.84" y2="83.82" width="0.1524" layer="91"/>
-<pinref part="JP2" gate="A" pin="1"/>
+<pinref part="UART" gate="A" pin="1"/>
 <wire x1="116.84" y1="83.82" x2="127" y2="83.82" width="0.1524" layer="91"/>
 </segment>
@@
 <wire x1="33.02" y1="116.84" x2="12.7" y2="116.84" width="0.1524" layer="91"/>
 <wire x1="12.7" y1="116.84" x2="12.7" y2="124.46" width="0.1524" layer="91"/>
-</segment>
-<segment>
-<pinref part="ISP1" gate="G$1" pin="VCC"/>
+<wire x1="12.7" y1="116.84" x2="12.7" y2="114.3" width="0.1524" layer="91"/>
+<junction x="12.7" y="116.84"/>
+<pinref part="J1" gate="JP1" pin="3.3V@17"/>
+<wire x1="12.7" y1="114.3" x2="33.02" y2="114.3" width="0.1524" layer="91"/>
+</segment>
+<segment>
+<pinref part="ISP" gate="G$1" pin="VCC"/>
 <pinref part="+3V2" gate="G$1" pin="+3V3"/>
 <wire x1="139.7" y1="121.92" x2="147.32" y2="121.92" width="0.1524" layer="91"/>
@@
 </segment>
 </net>
+<net name="MOSI" class="0">
+<segment>
+<pinref part="ISP" gate="G$1" pin="MOSI"/>
+<wire x1="147.32" y1="119.38" x2="139.7" y2="119.38" width="0.1524" layer="91"/>
+<label x="144.78" y="119.38" size="1.778" layer="95"/>
+</segment>
+<segment>
+<pinref part="J1" gate="JP1" pin="MOSI"/>
+<wire x1="73.66" y1="101.6" x2="63.5" y2="101.6" width="0.1524" layer="91"/>
+<label x="68.58" y="101.6" size="1.778" layer="95"/>
+</segment>
+<segment>
+<pinref part="SPI" gate="G$1" pin="3"/>
+<wire x1="109.22" y1="147.32" x2="99.06" y2="147.32" width="0.1524" layer="91"/>
+<label x="104.14" y="147.32" size="1.778" layer="95"/>
+</segment>
+</net>
+<net name="SCK" class="0">
+<segment>
+<pinref part="ISP" gate="G$1" pin="SCK"/>
+<wire x1="104.14" y1="119.38" x2="111.76" y2="119.38" width="0.1524" layer="91"/>
+<label x="104.14" y="119.38" size="1.778" layer="95"/>
+</segment>
+<segment>
+<pinref part="J1" gate="JP1" pin="SCLK"/>
+<wire x1="73.66" y1="106.68" x2="63.5" y2="106.68" width="0.1524" layer="91"/>
+<label x="68.58" y="106.68" size="1.778" layer="95"/>
+</segment>
+<segment>
+<pinref part="SPI" gate="G$1" pin="5"/>
+<wire x1="109.22" y1="152.4" x2="99.06" y2="152.4" width="0.1524" layer="91"/>
+<label x="104.14" y="152.4" size="1.778" layer="95"/>
+</segment>
+</net>
+<net name="MISO" class="0">
+<segment>
+<pinref part="ISP" gate="G$1" pin="MISO"/>
+<wire x1="104.14" y1="121.92" x2="111.76" y2="121.92" width="0.1524" layer="91"/>
+<label x="104.14" y="121.92" size="1.778" layer="95"/>
+</segment>
+<segment>
+<pinref part="J1" gate="JP1" pin="MISO"/>
+<wire x1="73.66" y1="104.14" x2="63.5" y2="104.14" width="0.1524" layer="91"/>
+<label x="68.58" y="104.14" size="1.778" layer="95"/>
+</segment>
+<segment>
+<pinref part="SPI" gate="G$1" pin="4"/>
+<wire x1="109.22" y1="149.86" x2="99.06" y2="149.86" width="0.1524" layer="91"/>
+<label x="104.14" y="149.86" size="1.778" layer="95"/>
+</segment>
+</net>
+<net name="RST" class="0">
+<segment>
+<pinref part="ISP" gate="G$1" pin="RST"/>
+<wire x1="104.14" y1="116.84" x2="111.76" y2="116.84" width="0.1524" layer="91"/>
+<label x="104.14" y="116.84" size="1.778" layer="95"/>
+</segment>
+<segment>
+<pinref part="J1" gate="JP1" pin="GP22"/>
+<wire x1="73.66" y1="83.82" x2="63.5" y2="83.82" width="0.1524" layer="91"/>
+<label x="68.58" y="83.82" size="1.778" layer="95"/>
+</segment>
+</net>
+<net name="SDA" class="0">
+<segment>
+<pinref part="J1" gate="JP1" pin="SDA"/>
+<wire x1="73.66" y1="121.92" x2="63.5" y2="121.92" width="0.1524" layer="91"/>
+<label x="68.58" y="121.92" size="1.778" layer="95"/>
+</segment>
+<segment>
+<pinref part="I2C" gate="G$1" pin="2"/>
+<wire x1="142.24" y1="149.86" x2="134.62" y2="149.86" width="0.1524" layer="91"/>
+<label x="137.16" y="149.86" size="1.778" layer="95"/>
+</segment>
+</net>
+<net name="SCL" class="0">
+<segment>
+<pinref part="J1" gate="JP1" pin="SCL"/>
+<wire x1="73.66" y1="119.38" x2="63.5" y2="119.38" width="0.1524" layer="91"/>
+<label x="68.58" y="119.38" size="1.778" layer="95"/>
+</segment>
+<segment>
+<pinref part="I2C" gate="G$1" pin="1"/>
+<wire x1="142.24" y1="147.32" x2="134.62" y2="147.32" width="0.1524" layer="91"/>
+<label x="137.16" y="147.32" size="1.778" layer="95"/>
+</segment>
+</net>
+<net name="CE0" class="0">
+<segment>
+<pinref part="J1" gate="JP1" pin="CE0"/>
+<wire x1="73.66" y1="99.06" x2="63.5" y2="99.06" width="0.1524" layer="91"/>
+<label x="68.58" y="99.06" size="1.778" layer="95"/>
+</segment>
+<segment>
+<pinref part="SPI" gate="G$1" pin="2"/>
+<wire x1="109.22" y1="144.78" x2="99.06" y2="144.78" width="0.1524" layer="91"/>
+<label x="104.14" y="144.78" size="1.778" layer="95"/>
+</segment>
+</net>
+<net name="CE1" class="0">
+<segment>
+<pinref part="J1" gate="JP1" pin="CE1"/>
+<wire x1="73.66" y1="96.52" x2="63.5" y2="96.52" width="0.1524" layer="91"/>
+<label x="68.58" y="96.52" size="1.778" layer="95"/>
+</segment>
+<segment>
+<pinref part="SPI" gate="G$1" pin="1"/>
+<wire x1="109.22" y1="142.24" x2="99.06" y2="142.24" width="0.1524" layer="91"/>
+<label x="104.14" y="142.24" size="1.778" layer="95"/>
+</segment>
+</net>
